File: Grove Button x2/Grove - Button x2.brd (EAGLE design)
At the start: 42.1 x 24.2 mm, 10 parts, among them J2 TWIG_2.0, SW1 DT6, SW2 DT6

Commit message: Help
Some help on board
Routing:
- net N$1: track 30.2 -> 33.5 mm, vias 1 -> 0
Other:
- board text added: "+"
- board text added: "Active state"
- board text added: "Standby state"
Changed lines of the file:
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@@
 <text x="8.89" y="2.2225" size="0.8128" layer="26" rot="MR0">hugo, 07/2015</text>
 <text x="12.3825" y="3.4925" size="0.8128" layer="26" rot="MR0">www.digitalspirit.org</text>
+<text x="18.415" y="15.875" size="0.8128" layer="26" rot="MR0">Active
+state</text>
+<wire x1="18.7325" y1="16.8275" x2="20.0025" y2="16.8275" width="0.127" layer="26"/>
+<wire x1="19.685" y1="17.145" x2="20.0025" y2="16.8275" width="0.127" layer="26"/>
+<wire x1="20.0025" y1="16.8275" x2="19.685" y2="16.51" width="0.127" layer="26"/>
+<wire x1="25.7175" y1="2.54" x2="27.6225" y2="2.54" width="0.127" layer="26"/>
+<wire x1="26.035" y1="2.8575" x2="25.7175" y2="2.54" width="0.127" layer="26"/>
+<wire x1="25.7175" y1="2.54" x2="26.035" y2="2.2225" width="0.127" layer="26"/>
+<wire x1="18.7325" y1="4.1275" x2="18.415" y2="3.4925" width="0.127" layer="26"/>
+<wire x1="18.415" y1="3.4925" x2="19.05" y2="3.4925" width="0.127" layer="26"/>
+<wire x1="18.415" y1="3.4925" x2="19.685" y2="4.445" width="0.127" layer="26"/>
+<wire x1="19.685" y1="4.445" x2="25.7175" y2="4.445" width="0.127" layer="26"/>
+<wire x1="25.7175" y1="4.445" x2="27.6225" y2="2.54" width="0.127" layer="26"/>
+<wire x1="27.6225" y1="2.54" x2="27.94" y2="2.54" width="0.127" layer="26"/>
+<text x="33.02" y="1.5875" size="0.8128" layer="26" rot="MR0">Standby
+state</text>
+<text x="21.9075" y="14.2875" size="1.27" layer="26" rot="MR0">+</text>
+<text x="13.0175" y="1.905" size="1.27" layer="26" rot="MR0">+</text>
+<text x="20.0025" y="1.905" size="1.27" layer="26" rot="MR0">+</text>
 </plain>
 <attributes>
@@
 <vertex x="-3.429" y="-3.937"/>
 </polygon>
-<via x="17.78" y="5.08" extent="1-16" drill="0.8128" diameter="1.27"/>
 </signal>
 <signal name="N$1">
@@
 <wire x1="26.67" y1="7.3025" x2="22.86" y2="7.3025" width="0.6096" layer="16"/>
 <wire x1="22.86" y1="7.3025" x2="22.86" y2="7.3" width="0.6096" layer="16"/>
-<wire x1="22.86" y1="9.8425" x2="22.86" y2="7.3" width="0.6096" layer="16"/>
 <contactref element="J2" pad="2"/>
-<wire x1="4.445" y1="10.779" x2="10.4935" y2="10.779" width="0.6096" layer="1"/>
-<wire x1="10.4935" y1="10.779" x2="11.43" y2="9.8425" width="0.6096" layer="1"/>
-<wire x1="11.43" y1="9.8425" x2="22.86" y2="9.8425" width="0.6096" layer="1"/>
-<via x="22.86" y="9.8425" extent="1-16" drill="0.8128" diameter="1.27"/>
+<wire x1="4.445" y1="10.779" x2="5.4135" y2="10.779" width="0.6096" layer="1"/>
+<wire x1="5.4135" y1="10.779" x2="6.35" y2="9.8425" width="0.6096" layer="1"/>
+<wire x1="6.35" y1="9.8425" x2="25.7175" y2="9.8425" width="0.6096" layer="1"/>
+<wire x1="25.7175" y1="9.8425" x2="26.67" y2="8.89" width="0.6096" layer="1"/>
+<wire x1="26.67" y1="8.89" x2="26.67" y2="7.3025" width="0.6096" layer="1"/>
 </signal>
 <signal name="N$2">
@@
 <wire x1="21.336" y1="16.8275" x2="21.336" y2="14.6685" width="0.6096" layer="16"/>
 <wire x1="21.336" y1="14.6685" x2="20.6375" y2="13.97" width="0.6096" layer="16"/>
-<wire x1="21.2725" y1="8.5725" x2="21.2725" y2="2.6035" width="0.6096" layer="16"/>
+<wire x1="21.2725" y1="9.8425" x2="21.2725" y2="2.6035" width="0.6096" layer="16"/>
 <wire x1="21.2725" y1="2.6035" x2="21.336" y2="2.54" width="0.6096" layer="16"/>
-<wire x1="20.6375" y1="13.97" x2="12.3825" y2="13.97" width="0.6096" layer="16"/>
-<wire x1="12.3825" y1="13.97" x2="11.7475" y2="13.335" width="0.6096" layer="16"/>
-<wire x1="11.7475" y1="13.335" x2="11.7475" y2="10.16" width="0.6096" layer="16"/>
-<wire x1="11.7475" y1="10.16" x2="12.3825" y2="9.525" width="0.6096" layer="16"/>
-<wire x1="12.3825" y1="9.525" x2="20.32" y2="9.525" width="0.6096" layer="16"/>
-<wire x1="20.32" y1="9.525" x2="21.2725" y2="8.5725" width="0.6096" layer="16"/>
+<wire x1="20.6375" y1="13.97" x2="12.7" y2="13.97" width="0.6096" layer="16"/>
+<wire x1="12.7" y1="13.97" x2="11.7475" y2="13.0175" width="0.6096" layer="16"/>
+<wire x1="11.7475" y1="13.0175" x2="11.7475" y2="11.7475" width="0.6096" layer="16"/>
+<wire x1="11.7475" y1="11.7475" x2="12.7" y2="10.795" width="0.6096" layer="16"/>
+<wire x1="12.7" y1="10.795" x2="20.32" y2="10.795" width="0.6096" layer="16"/>
+<wire x1="20.32" y1="10.795" x2="21.2725" y2="9.8425" width="0.6096" layer="16"/>
 <wire x1="13.6525" y1="4.445" x2="14.2875" y2="3.81" width="0.6096" layer="16"/>
 <wire x1="14.2875" y1="3.81" x2="14.2875" y2="2.6035" width="0.6096" layer="16"/>
@@
 </board>
 </drawing>
+<compatibility>
+<note version="6.3" minversion="6.2.2" severity="warning">
+Since Version 6.2.2 text objects can contain more than one line,
+which will not be processed correctly with this version.
+</note>
+</compatibility>
 </eagle>
